File: reader_hw/most_reader.kicad_pcb (KiCad board)
At the start: 2 copper layers, 77.5 x 55.5 mm, 62 parts, among them J1 1-1394640-1, J4 VBAT_IN, J6 PLT133/T10W, M1 Tang Nano 20K, U1 74LVC1G34, U3 74LVC1G125, U4 74LVC1G123, U5 TPS7B8133DRV, U6 LMR38020F

Commit message: J6: Everlight PLT237/T10WH on the same footprint; C32 1u; the fab package's PDFs
The PLT133/T10W the board was drawn for is out of production (Everlight's last time buy
2019-09-30, Rutronik; DigiKey has none and takes no backorder). The listener moved to
Cliff ORJ-5/OTJ-5 because its receiver went too; this board has none, and the PLT133's
successor in the same T10 housing, PLT237/T10WH (DPL-0000256 Rev.1), fits the footprint
as it is: pins 1 Vin, 2 Vcc, 3 GND on 2.54, pegs 1.10 on 5.08 2.62 typ in front of them
(the footprint's 2.63), 8.66 +-0.40 to the front foot (its 8.76). 2.7 to 5.0 V,
-40 to +85 C (the Cliff part: -20 to +70), 10 mm tall (19), 5.5 mA typical, 10 at most,
so FPGA pin 16 still feeds it: VCCIO - 0.4 V at least (DS226), 3.21 V by the IBIS model.
DigiKey 1080-PLT237/T10WH-ND; LCSC lists C17296340, none in stock on 2026-10-04. Only
J6's value and description change on the board; no copper moves.

C32 on 3V3_SW is 1u (C28323, a basic part), not 10u: pin 16 charges it at its
short-circuit current, about 0.18 A, when the FPGA starts, out of the module's 3.3 V
that also feeds VCCX and the SDRAM; 1u makes that pulse 30 us instead of 300.

make_fab.py now writes the schematic as a PDF and an assembly drawing of the top (every
reference, also the eight hidden on the silk), their dates pinned to the board's; the
committed reader_hw/most_reader.pdf was the step-2 sheet (no C83..C85, TP10, pin 16)
and goes. "3 mA" in the old notes was the PLT133's minimum. Sheet, ERC, DRC with
parity, pins and the fab package pass.

Co-Authored-By: Claude Opus 5.5 <noreply@anthropic.com>
Parts:
- C32: value 10u -> 1u
- J6: value PLT133/T10W -> PLT237/T10WH
Changed lines of the file:
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@@
 		(layer "F.Cu")
 		(at 68.776 20.5 90)
-		(descr "Everlight PLT133/T10W transmitter (the PLR135/T10 receiver's TOSLINK housing): 3 pins on 2.54, two pegs 2.63 in front of them, towards the optical port, which faces +y; the board's edge at the front foot, 8.76 in front of the pins, the port 2.35 past it; data sheet DPL-0000049 Rev.5 p.4")
-		(tags "TOSLINK Everlight PLT133 PLR135")
+		(descr "Everlight PLT237/T10WH transmitter (the T10 TOSLINK housing of PLT133/T10W and PLR135/T10): 3 pins on 2.54, two pegs 2.63 in front of them, towards the optical port, which faces +y; the board's edge at the front foot, 8.76 in front of the pins, the port 2.35 past it; data sheets DPL-0000256 Rev.1 p.4, DPL-0000049 Rev.5 p.4")
+		(tags "TOSLINK Everlight PLT237 PLT133")
 		(property "Reference" "J6"
 			(at -4 4.76 0)
@@
 			)
 		)
-		(property "Value" "PLT133/T10W"
+		(property "Value" "PLT237/T10WH"
 			(at 0 12.71 90)
 			(layer "F.Fab")
@@
 			)
 		)
-		(property "Value" "10u"
+		(property "Value" "1u"
 			(at 0 1.68 0)
 			(layer "F.Fab")
