File: reader_hw/most_reader.kicad_sch (KiCad schematic)
At the start: 54 parts, among them J1 1-1394640-1, J4 VBAT_IN, J6 PLT133/T10W, M1 Tang Nano 20K, U1 74LVC1G34, U3 74LVC1G125, U4 74LVC1G123, U5 TPS7B8133DRV, U6 LMR38020F

Commit message: Step 2, the board routed: the user's placement, 77.54 x 55.55 mm, no jumper
The layout is the board's own, not the listener's cut down. The user re-placed it six
times on 2026-10-03 and cut 6.45 mm off the top. gen_reader_pcb.py's PLACE, REFPOS and
TPTEXT now hold that placement, read back off the board, and --fresh on a copy lays
every part where the board has it.

Routing follows the listener's scheme. Every signal and supply runs on the top. The
bottom is one unbroken ground plane with nothing but vias in it. The top pour is
stitched every 6 mm, and every SMD ground pad has its own via.
- The ring: RXD 4 mm from J1 to R1/U1, TXD up a lane to J1 pin 1, RX_BUF through U1's
  and U3's bodies to the FPGA's pin 27, its branch to U4 between J1's pins 5 and 6.
- 3V3_AON from U5 under J1's body into FB2 and FB1.
- VBAT_P under the module to the buck.
- 5 V up the right edge to C63, C85, C64 and D3.
- No signal within 3.5 mm of a mounting hole's centre: TXD bends away from H1, S/PDIF
  goes round H2.

The sheet, from the user's edits:
- C83 (100 nF, 100 V) moves across the input behind F1, beside D2.
- C84 (100 V) on the VBAT_P riser.
- C85 on 5V_SW.
- TP10, a second ground test point.
- 3V3_SW, the supply of U3 and J6, now comes from module pin 7 (FPGA pin 16, LED1,
  held high by the gateware: U3 takes microamps, J6 3 mA, 10 at most), not pin 19.
  Pin 7 sits above /WAKE, so the last jumper is gone. The module's own 3.3 V pins are
  not wired.

The board carries a title block: JLR MOST reader, rev 1.0, 2026-10-03.

Checks: DRC 0 violations, 0 unconnected, 0 differences from the sheet. ERC 0/0.
check_sheet PASS. Tracks 558 mm, all on the top; 155 vias, all ground.

Co-Authored-By: Claude Opus 5.5 <noreply@anthropic.com>
Parts:
- added C83, C84: 100n 100V, Capacitor_SMD:C_0603_1608Metric, symbol Device:C
- added C85: 100n, Capacitor_SMD:C_0603_1608Metric, symbol Device:C
- added TP10: GND, TestPoint:TestPoint_Pad_D2.0mm, symbol Connector:TestPoint
Connections:
- net 3V3_SW: now also M1.7 (16 LED1); no longer M1.19 (3V3)
- net 5V_SW: now also C85.1
- net GND: now also C83.2, C84.2, C85.2, TP10.1
- net VBAT_P: now also C84.1
- net at D1.2 (A), D2.1 (K), F1.2: now also C83.1
Other:
- note added: "3V3_SW = вивід FPGA 16 (контакт 7, LED1) у постійній 1: U3 і J6. 3V3 модуля (19, 36) вільні: 3V3_SW не перетинає WAKE."
- note added: "5V_SW (U6, 80 В, 400 кГц) за WAKE: модуль FPGA, від його виводу 16 ще U3 і J6, ~0.3 А. L2 + C44/C45: 400 кГц не в джгут."
- note added: "C84 біля C45 (на платі)."
- note added: "D3: USB і 5V_SW разом не з'єднуються; U6 дає 5.3 В, на модулі ~5.0 В. Решта виводів вільна; логи - USB-UART модуля."
- note added: "SPDIF_F <- 42 (LCD_R3, IOB42B) через OSER8 на тій самій сітці; пара IOB42A у QN88 не виведена. Обидва лише на порожньому роз'ємі LCD."
- note added: "U3 від 3V3_SW: поки FPGA не працює,"
- note added: "Vcc передавача з 3V3_SW (вивід FPGA 16): 3 мА, до 10 мА (PLT133); C31/C32 біля J6. Корпус T10: виводи 8.5 мм від краю,"
- note removed: "5V_SW (U6, 80 В, 400 кГц) за WAKE: модуль FPGA, від його 3V3 ще U3 і J6, ~0.3 А. L2 + C44/C45: 400 кГц не в джгут."
- note removed: "D3: USB і 5V_SW разом не з'єднуються; U6 дає 5.3 В, на модулі ~5.0 В. 3V3_SW з модуля: U3, J6."
- note removed: "SPDIF_F <- 42 (LCD_R3) через OSER8 на тій самій сітці; 41 (його пара) вільний. Обидва лише на порожньому роз'ємі LCD."
- note removed: "U3 від 3V3_SW: коли FPGA вимкнена,"
- note removed: "Vcc передавача з 3V3_SW модуля: ~20 мА на світлодіод; C31/C32 біля J6. Корпус T10: виводи 8.5 мм від краю плати,"
- note removed: "Решта виводів вільна. Логи і запис кільця - через USB-UART самого модуля (BL616), стан - на його світлодіодах."

Commit message: J6: Everlight PLT237/T10WH on the same footprint; C32 1u; the fab package's PDFs
The PLT133/T10W the board was drawn for is out of production (Everlight's last time buy
2019-09-30, Rutronik; DigiKey has none and takes no backorder). The listener moved to
Cliff ORJ-5/OTJ-5 because its receiver went too; this board has none, and the PLT133's
successor in the same T10 housing, PLT237/T10WH (DPL-0000256 Rev.1), fits the footprint
as it is: pins 1 Vin, 2 Vcc, 3 GND on 2.54, pegs 1.10 on 5.08 2.62 typ in front of them
(the footprint's 2.63), 8.66 +-0.40 to the front foot (its 8.76). 2.7 to 5.0 V,
-40 to +85 C (the Cliff part: -20 to +70), 10 mm tall (19), 5.5 mA typical, 10 at most,
so FPGA pin 16 still feeds it: VCCIO - 0.4 V at least (DS226), 3.21 V by the IBIS model.
DigiKey 1080-PLT237/T10WH-ND; LCSC lists C17296340, none in stock on 2026-10-04. Only
J6's value and description change on the board; no copper moves.

C32 on 3V3_SW is 1u (C28323, a basic part), not 10u: pin 16 charges it at its
short-circuit current, about 0.18 A, when the FPGA starts, out of the module's 3.3 V
that also feeds VCCX and the SDRAM; 1u makes that pulse 30 us instead of 300.

make_fab.py now writes the schematic as a PDF and an assembly drawing of the top (every
reference, also the eight hidden on the silk), their dates pinned to the board's; the
committed reader_hw/most_reader.pdf was the step-2 sheet (no C83..C85, TP10, pin 16)
and goes. "3 mA" in the old notes was the PLT133's minimum. Sheet, ERC, DRC with
parity, pins and the fab package pass.

Co-Authored-By: Claude Opus 5.5 <noreply@anthropic.com>
Parts:
- C32: value 10u -> 1u
- J6: value PLT133/T10W -> PLT237/T10WH; symbol most_reader:PLT133 -> most_reader:PLT237
Other:
- note added: "SPDIF_F (FPGA 42) -> R28 -> J6 PLT237/T10WH: один вихід, лише TOSLINK (коаксіального J7 немає)."
- note added: "Vcc передавача з 3V3_SW (вивід FPGA 16): 5.5 мА типово, до 10 мА. C31 100n біля J6; C32 лише 1u: при старті"
- note added: "його заряджає ніжка FPGA. Корпус T10: виводи 8.76 мм від краю, лапка на краю, порт за краєм на 2.35 мм."
- note removed: "SPDIF_F (FPGA 42) -> R28 -> J6 PLT133/T10W: один вихід, лише TOSLINK (коаксіального J7 немає)."
- note removed: "Vcc передавача з 3V3_SW (вивід FPGA 16): 3 мА, до 10 мА (PLT133); C31/C32 біля J6. Корпус T10: виводи 8.5 мм від краю,"
- note removed: "лапка на краю, порт виступає на 2.6 мм (креслення Everlight, третій кут; перевірено в MOST25-to-AUDIO v1.4)."
Changed lines of the file:
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@@
   (pin "1") (pin "2")
   (instances (project "most_reader" (path "/344a96be-f3ba-5644-a956-0faca80b8b85" (reference "R28") (unit 1)))))
-(symbol (lib_id "most_reader:PLT133") (at 261.62 229.87 0) (unit 1) (exclude_from_sim no) (in_bom yes) (on_board yes) (dnp no)
+(symbol (lib_id "most_reader:PLT237") (at 261.62 229.87 0) (unit 1) (exclude_from_sim no) (in_bom yes) (on_board yes) (dnp no)
   (property "Reference" "J6" (at 254 222.25 0) (effects (font (size 1.27 1.27)) (justify left bottom)))
-  (property "Value" "PLT133/T10W" (at 270.51 229.87 0) (effects (font (size 1.27 1.27)) (justify left)))
+  (property "Value" "PLT237/T10WH" (at 270.51 229.87 0) (effects (font (size 1.27 1.27)) (justify left)))
   (property "Footprint" "most_reader:Everlight_TOSLINK_T10" (at 261.62 229.87 0) (effects (font (size 1.27 1.27)) (hide yes)))
   (property "Datasheet" "" (at 261.62 229.87 0) (effects (font (size 1.27 1.27)) (hide yes)))
@@
 (symbol (lib_id "Device:C") (at 281.94 218.44 0) (unit 1) (exclude_from_sim no) (in_bom yes) (on_board yes) (dnp no)
   (property "Reference" "C32" (at 284.48 217.17 0) (effects (font (size 1.27 1.27)) (justify left)))
-  (property "Value" "10u" (at 284.48 219.71 0) (effects (font (size 1.27 1.27)) (justify left)))
+  (property "Value" "1u" (at 284.48 219.71 0) (effects (font (size 1.27 1.27)) (justify left)))
   (property "Footprint" "Capacitor_SMD:C_0805_2012Metric" (at 281.94 218.44 0) (effects (font (size 1.27 1.27)) (hide yes)))
   (property "Datasheet" "" (at 281.94 218.44 0) (effects (font (size 1.27 1.27)) (hide yes)))
@@
   (pin "1")
   (instances (project "most_reader" (path "/344a96be-f3ba-5644-a956-0faca80b8b85" (reference "#PWR065") (unit 1)))))
-(text "SPDIF_F (FPGA 42) -> R28 -> J6 PLT133/T10W: один вихід, лише TOSLINK (коаксіального J7 немає)." (exclude_from_sim no) (at 212.09 242.57 0) (effects (font (size 1.27 1.27)) (justify left bottom)))
-(text "Vcc передавача з 3V3_SW (вивід FPGA 16): 3 мА, до 10 мА (PLT133); C31/C32 біля J6. Корпус T10: виводи 8.5 мм від краю," (exclude_from_sim no) (at 212.09 246.38 0) (effects (font (size 1.27 1.27)) (justify left bottom)))
-(text "лапка на краю, порт виступає на 2.6 мм (креслення Everlight, третій кут; перевірено в MOST25-to-AUDIO v1.4)." (exclude_from_sim no) (at 212.09 250.19 0) (effects (font (size 1.27 1.27)) (justify left bottom)))
+(text "SPDIF_F (FPGA 42) -> R28 -> J6 PLT237/T10WH: один вихід, лише TOSLINK (коаксіального J7 немає)." (exclude_from_sim no) (at 212.09 242.57 0) (effects (font (size 1.27 1.27)) (justify left bottom)))
+(text "Vcc передавача з 3V3_SW (вивід FPGA 16): 5.5 мА типово, до 10 мА. C31 100n біля J6; C32 лише 1u: при старті" (exclude_from_sim no) (at 212.09 246.38 0) (effects (font (size 1.27 1.27)) (justify left bottom)))
+(text "його заряджає ніжка FPGA. Корпус T10: виводи 8.76 мм від краю, лапка на краю, порт за краєм на 2.35 мм." (exclude_from_sim no) (at 212.09 250.19 0) (effects (font (size 1.27 1.27)) (justify left bottom)))
 (rectangle (start 335.28 203.2) (end 406.4 254) (stroke (width 0.254) (type dash) (color 72 72 160 1)) (fill (type none)))
 (text "7. ТЕСТОВІ ТОЧКИ" (exclude_from_sim no) (at 336.55 207.01 0) (effects (font (size 2 2) (bold yes)) (justify left bottom)))
