File: reader_hw2/most_reader_v2.kicad_sch (KiCad schematic)
At the start: 60 parts, among them J1 1-1394640-1, J4 VBAT_IN, J6 PLT237/T10WH, M1 Tang Nano 20K, U1 74LVC1G34, U3 74LVC1G125, U4 74LVC1G123, U5 TPS7B8133DRV, U6 LMR38020F

Commit message: reader v2.0: modernized - the board 84.9 mm, C45 8x10, the module on nine pins
The user re-placed the parts in KiCad round by round and the copper followed:
- power section: C6 between U6 and L1 (SW node 3.7 mm), C4 straight onto
  U6's VIN and exposed pad; C45 moved to the VBAT_P bus by U6
- C45 47u 63V in 8x10 (SamYoung MVK, C165628) instead of 100u 10x10.5, made
  in gen_reader2.py; check_v2_circuit allows exactly this change
- the module four header pins nearer J1, the board and tube 84.9 mm, J4 and
  J6 with the far edge; its footprint cut to nine pads (TANG_PINS)
- far end placed by the user: D3 lying with SPDIF between its pads, 3V3_SW
  from pin 7 between F1's and R28's pads; /WAKE and RX_BUF as diagonals
- 496 mm of copper (541), 75 vias (96), the same two top-layer hops

fab, caps, the kit READMEs and the READMEs regenerated for 84.9 mm.

Co-Authored-By: Claude Opus 5.5 <noreply@anthropic.com>
Parts:
- C45: value 100u 63V -> 47u 63V; footprint Capacitor_SMD:CP_Elec_10x10.5 -> Capacitor_SMD:CP_Elec_8x10
Other:
- note added: "решта знизу, J6 і J4 теж: під кінцем модуля з USB-C. У гребінці модуля лише контакти 5, 7, 8, 20, 21, 22, 25, 35, 40: решта ні до чого не йдуть."
- note removed: "решта знизу, J6 і J4 теж: під кінцем модуля з USB-C. Контакти 1..4 модуля під J4: у гребінку не ставляться."
Changed lines of the file:
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@@
 (kicad_sch (version 20231120) (generator "gen_reader") (generator_version "10.0") (paper "A3")
-(title_block (title "JLR MOST Reader v2.0: the board in a tube") (date "2026-10-05") (rev "2.0") (comment 1 "Generated by reader_hw2/gen_reader2.py from reader_hw/gen_reader.py: the circuit of v1.0 + R43, R44") (comment 2 "MOST25 bypass, an FPGA listening, S/PDIF out on TOSLINK, one clock"))
+(title_block (title "JLR MOST Reader v2.0: the board in a tube") (date "2026-10-05") (rev "2.0") (comment 1 "Generated by reader_hw2/gen_reader2.py from reader_hw/gen_reader.py: the circuit of v1.0 + R43, R44, C45 47u") (comment 2 "MOST25 bypass, an FPGA listening, S/PDIF out on TOSLINK, one clock"))
 (rectangle (start 12.7 12.7) (end 203.2 101.6) (stroke (width 0.254) (type dash) (color 72 72 160 1)) (fill (type none)))
 (text "1. ЖИВЛЕННЯ   J4 акумулятор -> 3V3_AON (завжди) і 5V_SW (за WAKE) -> модуль FPGA" (exclude_from_sim no) (at 13.97 16.51 0) (effects (font (size 2 2) (bold yes)) (justify left bottom)))
@@
 (symbol (lib_id "Device:C_Polarized") (at 57.15 67.31 0) (unit 1) (exclude_from_sim no) (in_bom yes) (on_board yes) (dnp no)
   (property "Reference" "C45" (at 54.61 66.04 0) (effects (font (size 1.27 1.27)) (justify right)))
-  (property "Value" "100u 63V" (at 54.61 68.58 0) (effects (font (size 1.27 1.27)) (justify right)))
-  (property "Footprint" "Capacitor_SMD:CP_Elec_10x10.5" (at 57.15 67.31 0) (effects (font (size 1.27 1.27)) (hide yes)))
+  (property "Value" "47u 63V" (at 54.61 68.58 0) (effects (font (size 1.27 1.27)) (justify right)))
+  (property "Footprint" "Capacitor_SMD:CP_Elec_8x10" (at 57.15 67.31 0) (effects (font (size 1.27 1.27)) (hide yes)))
   (property "Datasheet" "" (at 57.15 67.31 0) (effects (font (size 1.27 1.27)) (hide yes)))
   (pin "1") (pin "2")
@@
 (text "Що дасть лише запис у машині: яке з двох повідомлень гучності йде підсилювачу, крива байта 0x409, Connect." (exclude_from_sim no) (at 17.78 238.76 0) (effects (font (size 1.27 1.27)) (justify left bottom)))
 (text "v2.0: та сама схема на платі 26.5 мм у трубі 30x30x1.5. Зверху J1 і модуль (USB-C модуля в торцевій кришці)," (exclude_from_sim no) (at 17.78 242.57 0) (effects (font (size 1.27 1.27)) (justify left bottom)))
-(text "решта знизу, J6 і J4 теж: під кінцем модуля з USB-C. Контакти 1..4 модуля під J4: у гребінку не ставляться." (exclude_from_sim no) (at 17.78 246.38 0) (effects (font (size 1.27 1.27)) (justify left bottom)))
+(text "решта знизу, J6 і J4 теж: під кінцем модуля з USB-C. У гребінці модуля лише контакти 5, 7, 8, 20, 21, 22, 25, 35, 40: решта ні до чого не йдуть." (exclude_from_sim no) (at 17.78 246.38 0) (effects (font (size 1.27 1.27)) (justify left bottom)))
 (wire (pts (xy 17.78 129.54) (xy 27.94 129.54)) (stroke (width 0) (type default)))
 (wire (pts (xy 26.67 63.5) (xy 41.91 63.5)) (stroke (width 0) (type default)))
